File: DMH_SuperSaw_PANEL/DMH_SuperSaw_PANEL.kicad_pcb (KiCad board)
At the start: 2 copper layers, 100 x 200 mm, 29 parts, among them J0 Panel_GND_Solder_Wire_Pad

Commit message: Designed front panel
Parts:
- H10: value Env Amt -> F.E. Amt; footprint SynthStuff:Pot_Cutout_Tiny_attv_P110KH1 -> SynthStuff:Pot_Cutout_Small_attv_P110KH1
- H11: value Resonance -> Cutoff
- H12: value PWM CV -> Spread CV
- H13: value Attack -> Decay
- H14: value Decay -> Resonance
- H15: value Exp FM -> Cutoff CV
- H16: value Cutoff CV -> Exp CV
- H20: value Env Amt -> F.E. Amt
- H21, H8: value PWM -> Spread
- H23: value Sqr/Saw -> Oct 1
- H24: value LP/BP -> Oct 2
- H26: value AD/AR -> LP/BP
- H27: value Env/Drn -> A.E. +/d/-
- H5: value Coarse -> Attack
- H7: value Env Amt CV -> F.E. Amt CV
- H9: value Cutoff -> Sustain
Other:
- board text added: "2165"
- board text added: "Super Saw"
- board text removed: "2164"
- board text removed: "Sub Synth"

Commit message: Minor corrections
Parts:
- H13: value Decay -> Decay / Release
- H16: value Exp CV -> Exp FM CV
